Commit message: approach direction has been changed. now setting the robot ori to left

File: urdf/human/chest_included_npose.xacro (robot description, xacro)
@@ -16,5 +16,5 @@
     <parent link="world"/>
     <child link="base_link"/>
-    <origin rpy="0.0 0.0 0.0" xyz="0.0 -1.0 1.0"/>
+    <origin rpy="0.0 0.0 0.0" xyz="0 0 1.05"/>
   </joint>
   <link name="base_link">

Commit message: LW axis angle directions fixed, xacro LW revolute (not fixed anymore)

File: urdf/human/chest_included_npose.xacro (robot description, xacro)
@@ -311,12 +311,12 @@
     <limit effort="1" lower="0.0" upper="1.57079632679" velocity="1"/>
   </joint>
-  <joint name="left_wrist_0" type="fixed">
+  <joint name="left_wrist_0" type="revolute">
     <origin rpy="0 0 0" xyz="0.274149473988 0 0"/>
-    <axis xyz="0 -1 0"/>
+    <axis xyz="0 1 0"/>
     <parent link="human/left_elbow"/>
     <child link="human/left_wrist_0"/>
     <limit effort="1" lower="-0.78539816339" upper="0.78539816339" velocity="1"/>
   </joint>
-  <joint name="left_wrist_1" type="fixed">
+  <joint name="left_wrist_1" type="revolute">
     <origin rpy="0 0 0" xyz="0 0 0"/>
     <axis xyz="0 0 1"/>
@@ -325,5 +325,5 @@
     <limit effort="1" lower="-1.57079632679" upper="1.57079632679" velocity="1"/>
   </joint>
-  <joint name="left_wrist_2" type="fixed">
+  <joint name="left_wrist_2" type="revolute">
     <origin rpy="0 0 0" xyz="0 0 0"/>
     <axis xyz="1 0 0"/>
